File: hardware/SortingHat.sch (EAGLE design)
At the start: 26 parts, among them IC1 LM386MMX-1, J1 BATT, J2 SPKR, J3 RAND, U1 3.3V/150mA, U2 DYNASTREAM_N5150M4CD

Commit message: Version 1 of the PCB
This is the design as I sent it off to OSHPark.
Parts:
- added C10: 0.1uF, rcl:C-USC0805
- C6: device rcl:CPOL-USUD-4X5,8 -> SparkFun-Capacitors:10UF-POLAR-EIA3216-16V-10%(TANT)
- C7: value 10'uF -> 10uF; device rcl:CPOL-USUD-4X5,8 -> SparkFun-Capacitors:10UF-POLAR-EIA3216-16V-10%(TANT)
- C9: device rcl:CPOL-USUD-8X10 -> SparkFun-Capacitors:68UF-POLAR-EIA3528-10V-10%(TANT)
- J4: value (none) -> SERVO
- S1: value (none) -> POWER
- U2: value DYNASTREAM_N5150M4CD -> DYNASTREAM_N5150M4CDTOP; device adam_custom:DYNASTREAM_N5150M4CD -> adam_custom:DYNASTREAM_N5150M4CDTOP
Connections:
- net 5V: now also C10.1
- net GND: now also C10.2
- net MOUTH_SERVO: now also U2.P6; no longer U2.P2
- net RANDOM_SWITCH: now also U2.P8; no longer U2.P3
- net SDC_CS: now also U2.P2; no longer U2.P15
- net SDC_MISO: now also U2.P0; no longer U2.P24
- net SOUND: now also U2.P15; no longer U2.P0
Changed lines of the file:
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@@
 <parts>
 <part name="J1" library="SparkFun-Connectors" deviceset="CONN_02" device="1X02_NO_SILK" value="BATT"/>
-<part name="S1" library="adafruit" deviceset="EG1218" device="S"/>
+<part name="S1" library="adafruit" deviceset="EG1218" device="S" value="POWER"/>
 <part name="U1" library="SparkFun-IC-Power" deviceset="V_REG_MIC5205" device="3.3V" value="3.3V/150mA"/>
 <part name="GND1" library="SparkFun-PowerSymbols" deviceset="GND" device=""/>
@@
 <part name="GND3" library="SparkFun-PowerSymbols" deviceset="GND" device=""/>
 <part name="SUPPLY2" library="SparkFun-PowerSymbols" deviceset="3.3V" device=""/>
-<part name="U2" library="adam_custom" deviceset="DYNASTREAM_N5150M4CD" device=""/>
+<part name="U2" library="adam_custom" deviceset="DYNASTREAM_N5150M4CD" device="TOP"/>
 <part name="SUPPLY3" library="SparkFun-PowerSymbols" deviceset="3.3V" device=""/>
 <part name="GND4" library="SparkFun-PowerSymbols" deviceset="GND" device=""/>
@@
 <part name="C4" library="rcl" deviceset="C-US" device="C0805" value="0.1uF"/>
 <part name="C5" library="rcl" deviceset="C-US" device="C0805" value="0.01uF"/>
-<part name="C6" library="rcl" deviceset="CPOL-US" device="UD-4X5,8" value="10uF"/>
+<part name="C6" library="SparkFun-Capacitors" deviceset="10UF-POLAR" device="-EIA3216-16V-10%(TANT)" value="10uF"/>
 <part name="R5" library="pot" deviceset="TRIM_US-" device="3223W" value="10kΩ"/>
 <part name="GND5" library="SparkFun-PowerSymbols" deviceset="GND" device=""/>
 <part name="IC1" library="linear" deviceset="LM386?-*" device="MM" technology="1" value="LM386MMX-1"/>
 <part name="GND6" library="SparkFun-PowerSymbols" deviceset="GND" device=""/>
-<part name="C7" library="rcl" deviceset="CPOL-US" device="UD-4X5,8" value="10'uF"/>
+<part name="C7" library="SparkFun-Capacitors" deviceset="10UF-POLAR" device="-EIA3216-16V-10%(TANT)" value="10uF"/>
 <part name="SUPPLY4" library="SparkFun-PowerSymbols" deviceset="5V" device=""/>
 <part name="C8" library="rcl" deviceset="C-US" device="C0805" value="0.1uF"/>
 <part name="R6" library="rcl" deviceset="R-US_" device="R0805" value="10Ω"/>
-<part name="C9" library="rcl" deviceset="CPOL-US" device="UD-8X10" value="220uF"/>
+<part name="C9" library="SparkFun-Capacitors" deviceset="68UF-POLAR" device="-EIA3528-10V-10%(TANT)" value="220uF"/>
 <part name="GND7" library="SparkFun-PowerSymbols" deviceset="GND" device=""/>
 <part name="J2" library="SparkFun-Connectors" deviceset="CONN_02" device="1X02_NO_SILK" value="SPKR"/>
@@
 <part name="R7" library="rcl" deviceset="R-US_" device="R0805" value="1kΩ"/>
 <part name="SUPPLY6" library="SparkFun-PowerSymbols" deviceset="3.3V" device=""/>
-<part name="J4" library="SparkFun-Connectors" deviceset="CONN_03" device="1X03_NO_SILK"/>
+<part name="J4" library="SparkFun-Connectors" deviceset="CONN_03" device="1X03_NO_SILK" value="SERVO"/>
 <part name="SUPPLY7" library="SparkFun-PowerSymbols" deviceset="5V" device=""/>
 <part name="GND10" library="SparkFun-PowerSymbols" deviceset="GND" device=""/>
@@
 <attribute name="REV" value="1"/>
 </part>
+<part name="C10" library="rcl" deviceset="C-US" device="C0805" value="0.1uF"/>
+<part name="GND11" library="SparkFun-PowerSymbols" deviceset="GND" device=""/>
 </parts>
 <sheets>
@@
 <instances>
 <instance part="J1" gate="G$1" x="20.32" y="111.76"/>
-<instance part="S1" gate="1" x="35.56" y="116.84" rot="R270"/>
+<instance part="S1" gate="1" x="35.56" y="116.84" smashed="yes" rot="R270">
+<attribute name="NAME" x="33.655" y="123.19" size="1.778" layer="95"/>
+<attribute name="VALUE" x="31.877" y="108.712" size="1.778" layer="96"/>
+</instance>
 <instance part="U1" gate="U1" x="66.04" y="111.76"/>
 <instance part="GND1" gate="1" x="27.94" y="106.68"/>
@@
 <instance part="GND6" gate="1" x="182.88" y="88.9"/>
 <instance part="C7" gate="G$1" x="177.8" y="101.6"/>
-<instance part="SUPPLY4" gate="G$1" x="185.42" y="121.92"/>
+<instance part="SUPPLY4" gate="G$1" x="185.42" y="129.54"/>
 <instance part="C8" gate="G$1" x="210.82" y="104.14"/>
 <instance part="R6" gate="G$1" x="210.82" y="88.9" rot="R90"/>
@@
 <instance part="FRAME1" gate="G$1" x="0" y="0"/>
 <instance part="FRAME1" gate="V" x="147.32" y="0"/>
+<instance part="C10" gate="G$1" x="193.04" y="124.46" rot="R90"/>
+<instance part="GND11" gate="1" x="200.66" y="119.38"/>
 </instances>
 <busses>
@@
 <wire x1="187.96" y1="63.5" x2="187.96" y2="53.34" width="0.1524" layer="91"/>
 </segment>
+<segment>
+<pinref part="C10" gate="G$1" pin="2"/>
+<pinref part="GND11" gate="1" pin="GND"/>
+<wire x1="198.12" y1="124.46" x2="200.66" y2="124.46" width="0.1524" layer="91"/>
+<wire x1="200.66" y1="124.46" x2="200.66" y2="121.92" width="0.1524" layer="91"/>
+</segment>
 </net>
 <net name="N$1" class="0">
@@
 <pinref part="SUPPLY4" gate="G$1" pin="5V"/>
 <pinref part="IC1" gate="G$1" pin="VS"/>
-<wire x1="185.42" y1="121.92" x2="185.42" y2="119.38" width="0.1524" layer="91"/>
+<wire x1="185.42" y1="129.54" x2="185.42" y2="124.46" width="0.1524" layer="91"/>
+<pinref part="C10" gate="G$1" pin="1"/>
+<wire x1="185.42" y1="124.46" x2="185.42" y2="119.38" width="0.1524" layer="91"/>
+<wire x1="190.5" y1="124.46" x2="185.42" y2="124.46" width="0.1524" layer="91"/>
+<junction x="185.42" y="124.46"/>
 </segment>
 <segment>
@@
 <net name="SOUND" class="0">
 <segment>
-<pinref part="U2" gate="G$1" pin="P0"/>
-<wire x1="55.88" y1="88.9" x2="58.42" y2="88.9" width="0.1524" layer="91"/>
-<label x="58.42" y="88.9" size="1.016" layer="95" xref="yes"/>
-</segment>
-<segment>
 <pinref part="R1" gate="G$1" pin="1"/>
 <wire x1="114.3" y1="119.38" x2="111.76" y2="119.38" width="0.1524" layer="91"/>
 <label x="111.76" y="119.38" size="1.016" layer="95" rot="R180" xref="yes"/>
 </segment>
+<segment>
+<pinref part="U2" gate="G$1" pin="P15"/>
+<wire x1="55.88" y1="66.04" x2="58.42" y2="66.04" width="0.1524" layer="91"/>
+<label x="58.42" y="66.04" size="1.016" layer="95" xref="yes"/>
+</segment>
 </net>
 <net name="MOUTH_SERVO" class="0">
-<segment>
-<pinref part="U2" gate="G$1" pin="P2"/>
-<wire x1="55.88" y1="86.36" x2="58.42" y2="86.36" width="0.1524" layer="91"/>
-<label x="58.42" y="86.36" size="1.016" layer="95" xref="yes"/>
-</segment>
 <segment>
 <pinref part="J4" gate="J$1" pin="3"/>
@@
 <label x="185.42" y="58.42" size="1.016" layer="95" rot="R180" xref="yes"/>
 </segment>
+<segment>
+<pinref part="U2" gate="G$1" pin="P6"/>
+<wire x1="55.88" y1="78.74" x2="58.42" y2="78.74" width="0.1524" layer="91"/>
+<label x="58.42" y="78.74" size="1.016" layer="95" xref="yes"/>
+</segment>
 </net>
 <net name="RANDOM_SWITCH" class="0">
-<segment>
-<pinref part="U2" gate="G$1" pin="P3"/>
-<wire x1="55.88" y1="83.82" x2="58.42" y2="83.82" width="0.1524" layer="91"/>
-<label x="58.42" y="83.82" size="1.016" layer="95" xref="yes"/>
-</segment>
 <segment>
 <pinref part="J3" gate="G$1" pin="1"/>
@@
 <junction x="154.94" y="60.96"/>
 </segment>
+<segment>
+<pinref part="U2" gate="G$1" pin="P8"/>
+<wire x1="55.88" y1="76.2" x2="58.42" y2="76.2" width="0.1524" layer="91"/>
+<label x="58.42" y="76.2" size="1.016" layer="95" xref="yes"/>
+</segment>
 </net>
 <net name="SDC_CS" class="0">
-<segment>
-<pinref part="U2" gate="G$1" pin="P15"/>
-<wire x1="55.88" y1="66.04" x2="58.42" y2="66.04" width="0.1524" layer="91"/>
-<label x="58.42" y="66.04" size="1.016" layer="95" xref="yes"/>
-</segment>
 <segment>
 <pinref part="JP1" gate="G$1" pin="CS"/>
@@
 <label x="111.76" y="86.36" size="1.016" layer="95" rot="R180" xref="yes"/>
 </segment>
+<segment>
+<pinref part="U2" gate="G$1" pin="P2"/>
+<wire x1="55.88" y1="86.36" x2="58.42" y2="86.36" width="0.1524" layer="91"/>
+<label x="58.42" y="86.36" size="1.016" layer="95" xref="yes"/>
+</segment>
 </net>
 <net name="SDC_MOSI" class="0">
@@
 <net name="SDC_MISO" class="0">
 <segment>
-<pinref part="U2" gate="G$1" pin="P24"/>
-<wire x1="55.88" y1="60.96" x2="58.42" y2="60.96" width="0.1524" layer="91"/>
-<label x="58.42" y="60.96" size="1.016" layer="95" xref="yes"/>
-</segment>
-<segment>
 <pinref part="JP1" gate="G$1" pin="DO"/>
 <wire x1="114.3" y1="73.66" x2="111.76" y2="73.66" width="0.1524" layer="91"/>
 <label x="111.76" y="73.66" size="1.016" layer="95" rot="R180" xref="yes"/>
 </segment>
-</net>
+<segment>
+<pinref part="U2" gate="G$1" pin="P0"/>
+<wire x1="55.88" y1="88.9" x2="58.42" y2="88.9" width="0.1524" layer="91"/>
+<label x="58.42" y="88.9" size="1.016" layer="95" xref="yes"/>
+</segment>
+</net>
